File: Projects/KiCad/45-1599-1 tester/45-1599-1 PCB/45-1599-1 PCB/45-1599-1 PCB.kicad_pcb (KiCad board)
At the start: 2 copper layers, 388.6 x 236.2 mm, 47 parts, among them J1 CONN_01X14, J12 CONN_01X14, J13 CONN_01X14, J14 CONN_01X02_MALE, J15 CONN_01X06, J16 CONN_01X06, J17 CONN_01X08, J18 12V INPUT MAIN POWER, J19 Fan, J2 CONN_01X14, J3 CONN_01X14, J4 CONN_01X14, J5 CONN_01X14, J6 CONN_01X06, J8 CONN_01X14, J9 CONN_01X14, K1 EC2-5NU, K2 EC2-5NU, K3 EC2-5NU, K4 EC2-5NU, K5 EC2-5NU, K6 RT314A05, K7 RT314A05, SW1 SWITCH, U2 ARDUINO_NANO, U3 LM2576

Commit message: renewed
renewed
Parts:
- C1: value 100uF -> (none)
- C2: value 1000uF -> (none)
- D1, D10, D6, D9: value LED -> (none)
- D2, D3, D4, D5, D8: value D -> (none)
- D7: value D_Schottky -> (none)
- J12, J5: value CONN_01X14 -> (none); footprint Conn_02x07:2X8 -> ARDUINO_NANO_New:2X7
- J13: value CONN_01X14 -> (none)
- J14: value CONN_01X02_MALE -> (none); footprint Connector_PinHeader_2.00mm:PinHeader_1x02_P2.00mm_Vertical -> Connector_PinSocket_2.54mm new:PinSocket_1x02_P2.54mm_Vertical
- J15, J16, J6: value CONN_01X06 -> (none); footprint 2x3:2X8 -> ARDUINO_NANO_New:2X3
- J17: value CONN_01X08 -> (none); footprint 2x4:2X8 -> ARDUINO_NANO_New:2X4
- J18: value 12V INPUT MAIN POWER -> (none)
- J20: renamed from SW1; value SWITCH -> (none)
- K1, K2, K3, K4, K5: value EC2-5NU -> (none)
- K6, K7: value RT314A05 -> (none)
- L1: value L -> (none)
- Mega1: footprint Arduino Mega:Arduino_Mega2560_Shield -> ARDUINO_NANO_New:Arduino_Mega2560_Shield
- R1, R2, R4, R5: value R -> (none)
- R3: value 10K -> (none)
- R6: renamed from 3K1; value RESISTOR -> R6
- R7: renamed from 1K1; value RESISTOR -> R7
- U2: value ARDUINO_NANO -> (none)
- U3: value LM2576 -> (none)
- moved D7 185.2 mm to (424.2, 122.1), turned to 270 degrees
- moved C2 173.6 mm to (438.0, 125.3)
- moved C1 166.8 mm to (438.0, 141.7)
- moved U3 162.7 mm to (421.4, 160.9), turned to 180 degrees
- moved L1 149.4 mm to (422.5, 143.4)
- moved K6 50.1 mm to (414.2, 86.8), turned to 270 degrees
- moved J18 42.8 mm to (449.0, 295.0), turned to 90 degrees
- moved J14 39.3 mm to (441.0, 295.0), turned to 90 degrees
- moved D4 32.8 mm to (417.4, 293.8), turned to 270 degrees
- moved R7 31.9 mm to (437.0, 286.2), turned to 90 degrees
- moved K4 29.1 mm to (327.0, 94.0), turned to 180 degrees
- moved D2 28.3 mm to (401.4, 293.8), turned to 270 degrees
- moved R6 26.5 mm to (430.0, 286.2), turned to 90 degrees
- moved D3 25.7 mm to (409.4, 293.8), turned to 270 degrees
- moved R1 24.6 mm to (395.0, 286.2), turned to 90 degrees
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Routing:
- net 36Digital48_J4.1: track 558.0 -> 728.4 mm, vias 2 -> 6
- net +12VDC: track 194.5 -> 263.0 mm
- net Net-(J1-Pad10): track 434.3 -> 489.5 mm, vias 5 -> 2
- net Net-(J1-Pad2): track 416.4 -> 470.1 mm, vias 3 -> 5
- net Net-(J14-Pad1): track 261.2 -> 209.8 mm, vias 1 -> 0
- net Net-(J1-Pad3): track 457.9 -> 506.3 mm, vias 6 -> 7
- net Net-(D10-Pad2): track 298.6 -> 346.1 mm, vias 4 -> 3
- net 35Digital49_J18.1: track 543.2 -> 496.6 mm
- net Net-(J1-Pad5): track 484.9 -> 524.2 mm, vias 4 -> 8
- net +5VDC: track 279.1 -> 239.9 mm, vias 1 -> 2
- net J4.1: track 80.4 -> 115.5 mm, vias 1 -> 0
- net Net-(D9-Pad2): track 301.1 -> 335.6 mm, vias 2 -> 3
- net nanoDigital2: track 103.0 -> 71.4 mm
- net voltagDividerAnalogCheck: track 272.7 -> 302.5 mm, vias 0 -> 1
- net J4.2: track 80.6 -> 109.4 mm, vias 1 -> 0
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Other:
- copper layers 2 -> 4
- net class Default: clearance 0.2 -> 0.4
- rule trace_clearance: 0.2 -> 0.4
- board text added: "45-1569-1"
- board text added: "45-1603-1"
- board text added: "45-1613-1"
- board text added: "Arduino Mega"
- board text added: "Arduino Nano"
- board text added: "Hunter Engineering 45-1599-1 Functional Test PCB REV. B"
- board text added: "XILINX"
- board text removed: "45-1599-1 FUNCTIONAL TEST"
- board text removed: "Voltage Divider, R1 = 3k, R2 = 1k ratio of 3:1"
