File: Projects/KiCad/FINAL lm324m_Line/lm324m_Line/lm324_line.kicad_pcb (KiCad board)
At the start: 2 copper layers, 53.3 x 54.6 mm, 24 parts, among them J1 CONN_01X02_MALE, J2 CONN_01X02_MALE, J3 CONN_01X02_MALE, J4 CONN_01X02_MALE, J5 Screw_Terminal_1x02, K1 EC2-5NU, K2 EC2-5NU, Q1 2N3904, Q2 2N3904, U1 lm324

Commit message: renewed
renewed
Parts:
- added 0.1uf1: CP, Capacitors_THT:CP_Radial_D10.0mm_P5.00mm, F.Cu at (65.6, 93.0)
- added ?: , Mounting_Holes:MountingHole_3.2mm_M3, F.Cu at (120.2, 169.9)
- added ?: , Mounting_Holes:MountingHole_3.2mm_M3, F.Cu at (45.1, 169.5)
- added ?: , Mounting_Holes:MountingHole_3.2mm_M3, F.Cu at (120.1, 64.8)
- added ?: , Mounting_Holes:MountingHole_3.2mm_M3, F.Cu at (45.3, 65.6)
- added F1: , lm324m_Line:C320C, F.Cu at (46.1, 83.0)
- added J6: , Connector_PinHeader_2.54mm new:PinHeader_1x03_P2.54mm_Vertical, F.Cu at (52.0, 69.0)
- added J7: 9V+, Connector_PinHeader_2.54mm new:PinHeader_1x02_P2.54mm_Vertical, F.Cu at (52.0, 83.0)
- added J8: , Connector_PinHeader_2.54mm new:PinHeader_1x04_P2.54mm_Vertical, F.Cu at (53.0, 155.7)
- added TB1: ARDUINO_NANO, SHIELD_ARDUINO_NANO, F.Cu at (72.0, 113.0)
- added U2: AMS1117-5.0, Package_TO_SOT_Packages_THT:TO-126_Vertical, F.Cu at (51.8, 97.0)
- added U3: L293D, DIP880W50P254L2000H510Q16, F.Cu at (104.0, 128.2)
- D1, D2: value 1N4001 -> (none); footprint Diodes_THT:D_DO-41_SOD81_P12.70mm_Horizontal -> Diode_THT:D_DO-15_P15.24mm_Horizontal
- D3, D4: footprint LEDs:LED_D3.0mm -> LEDs:LED_D4.0mm
- J1, J2, J3, J4: value CONN_01X02_MALE -> (none); footprint 2 pin male connector:2_pin_male_connector -> Connector_PinHeader_2.54mm new:PinHeader_1x03_P2.54mm_Vertical
- J5: value Screw_Terminal_1x02 -> (none); footprint Connectors_Terminal_Blocks:TerminalBlock_bornier-2_P5.08mm -> Connector_PinHeader_2.54mm new:PinHeader_1x02_P2.54mm_Vertical
- K1, K2: value EC2-5NU -> (none)
- Q1, Q2: value 2N3904 -> (none); footprint 2N3904:TO92127P495H495-3 -> TO_SOT_Packages_THT:TO-92_Inline_Wide
- R1, R2: value 1k -> 10k; footprint Resistors_THT:R_Axial_DIN0204_L3.6mm_D1.6mm_P7.62mm_Horizontal -> Potentiometers:Potentiometer_Trimmer_ACP_CA6v_Horizontal
- R10: value 470 -> 470R; footprint Resistors_THT:R_Axial_DIN0204_L3.6mm_D1.6mm_P7.62mm_Horizontal -> Resistors_THT:R_Axial_DIN0309_L9.0mm_D3.2mm_P20.32mm_Horizontal
- R3: footprint Resistors_THT:R_Axial_DIN0207_L6.3mm_D2.5mm_P7.62mm_Horizontal -> Resistors_THT:R_Axial_DIN0309_L9.0mm_D3.2mm_P20.32mm_Horizontal
- R4: value 270 -> (none); footprint Resistors_THT:R_Axial_DIN0207_L6.3mm_D2.5mm_P7.62mm_Horizontal -> Resistors_THT:R_Axial_DIN0309_L9.0mm_D3.2mm_P20.32mm_Horizontal
- R5, R6: value 10k -> 1k; footprint pot:TRIM_3266W-1-103LF -> Resistors_THT:R_Axial_DIN0309_L9.0mm_D3.2mm_P20.32mm_Horizontal
- R7: footprint Resistors_THT:R_Axial_DIN0204_L3.6mm_D1.6mm_P7.62mm_Horizontal -> Resistors_THT:R_Axial_DIN0309_L9.0mm_D3.2mm_P20.32mm_Horizontal
- R8: value 10k -> 470R; footprint Resistors_THT:R_Axial_DIN0204_L3.6mm_D1.6mm_P7.62mm_Horizontal -> Resistors_THT:R_Axial_DIN0309_L9.0mm_D3.2mm_P20.32mm_Horizontal
- R9: value 470 -> 10k; footprint Resistors_THT:R_Axial_DIN0204_L3.6mm_D1.6mm_P7.62mm_Horizontal -> Resistors_THT:R_Axial_DIN0309_L9.0mm_D3.2mm_P20.32mm_Horizontal
- moved J5 91.8 mm to (52.0, 90.0), turned to 90 degrees
- moved R3 89.3 mm to (64.2, 162.0), turned to 0 degrees
- moved R10 88.9 mm to (64.4, 69.0), turned to 0 degrees
- moved J2 70.2 mm to (53.0, 162.0), turned to 90 degrees
- moved Q2 68.5 mm to (72.0, 146.6), turned to 90 degrees
- moved D4 67.3 mm to (52.0, 140.4), turned to 0 degrees
- moved J4 64.8 mm to (60.0, 141.0), turned to 90 degrees
- moved U1 63.6 mm to (104.0, 88.1)
- moved R9 63.3 mm to (110.3, 69.0), turned to 180 degrees
- moved J1 61.8 mm to (60.0, 153.0), turned to 90 degrees
- moved Q1 60.2 mm to (72.0, 134.7), turned to 90 degrees
- moved J3 59.1 mm to (60.0, 129.0), turned to 90 degrees
- moved R1 53.5 mm to (76.6, 97.0), turned to 0 degrees
- moved D3 52.7 mm to (52.0, 129.6), turned to 0 degrees
- moved R4 51.2 mm to (89.7, 162.0), turned to 0 degrees
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Connections:
- D1 pad 1: Net-(D1-Pad1) -> V+
- D2 pad 1: Net-(D2-Pad1) -> V+
- D3 pad 1: OutputPIN4 -> OutputPIN1
- D4 pad 1: OutputPIN1 -> OutputPIN4
- J1 pad 1: Net-(J1-Pad1) -> V+
- J2 pad 1: Net-(J2-Pad1) -> V+
- J2 pad 2: Input1- -> Net-(J2-Pad2)
- J3 pad 1: Net-(J2-Pad1) -> Motor1a
- J3 pad 2: Input1- -> Motor1b
- J4 pad 1: Net-(J4-Pad1) -> Motor2a
- J4 pad 2: Net-(J4-Pad2) -> Motor2b
- J5 pad 1: GND -> +9V
- J5 pad 2: V+ -> GND
- K1 pad 1: Net-(D1-Pad1) -> V+
- K1 pad 10: Net-(K1-Pad10) -> (no net)
- K1 pad 3: Net-(K1-Pad3) -> (no net)
- K1 pad 4: Net-(J1-Pad1) -> Motor2a
- K1 pad 5: Net-(J1-Pad2) -> Motor2b
- K1 pad 8: Net-(K1-Pad8) -> (no net)
- K1 pad 9: Net-(K1-Pad9) -> (no net)
- K2 pad 1: Net-(D2-Pad1) -> V+
- K2 pad 10: Net-(K2-Pad10) -> (no net)
- K2 pad 3: Net-(K2-Pad3) -> (no net)
- K2 pad 4: Net-(J4-Pad1) -> Motor1a
- K2 pad 5: Net-(J4-Pad2) -> Motor1b
- K2 pad 8: Net-(K2-Pad8) -> (no net)
- K2 pad 9: Net-(K2-Pad9) -> (no net)
- R1 pad 1: OutputPIN4 -> GND
- R1 pad 2: Net-(Q1-Pad2) -> Net-(J1-Pad2)
- R10 pad 2: Input4+ -> GND
- R2 pad 1: OutputPIN1 -> GND
- R2 pad 2: Net-(Q2-Pad2) -> Net-(J2-Pad2)
- R5 pad 1: Input4+ -> OutputPIN1
- R5 pad 2: Net-(J2-Pad1) -> Net-(Q1-Pad2)
- R6 pad 1: Input1+ -> OutputPIN4
- R6 pad 2: Net-(J2-Pad1) -> Net-(Q2-Pad2)
- R7 pad 1: Input1- -> V+
- R7 pad 2: V+ -> Input4-
- R8 pad 2: Input1- -> GND
- R9 pad 1: Input1+ -> V+
- R9 pad 2: V+ -> Input1-
- U1 pad 10: Net-(U1-Pad10) -> (no net)
- U1 pad 12: Input4+ -> GND
- U1 pad 13: Input1- -> Input4-
- U1 pad 3: Input1+ -> GND
- U1 pad 5: Net-(U1-Pad5) -> (no net)
- U1 pad 6: Net-(U1-Pad6) -> (no net)
- U1 pad 7: Net-(U1-Pad7) -> (no net)
- U1 pad 8: Net-(U1-Pad8) -> (no net)
- U1 pad 9: Net-(U1-Pad9) -> (no net)
Routing:
- net Input1-: track 161.8 -> 0.00 mm, vias 6 -> 0
- net GND: track 103.7 -> 0.00 mm, vias 2 -> 0
- net Net-(J2-Pad1): track 83.8 -> 0.00 mm, vias 2 -> 0
- net Input4+: track 67.3 -> 0.00 mm, vias 5 -> 0
- net OutputPIN1: track 61.9 -> 0.00 mm, vias 3 -> 0
- net OutputPIN4: track 47.7 -> 0.00 mm
- net V+: track 44.7 -> 0.00 mm, vias 1 -> 0
- net Net-(D3-Pad2): track 39.4 -> 0.00 mm
- net Net-(D1-Pad2): track 30.0 -> 0.00 mm
- net Input1+: track 26.4 -> 0.00 mm
- net Net-(D2-Pad2): track 21.9 -> 0.00 mm
- net Net-(D4-Pad2): track 21.8 -> 0.00 mm
- net Net-(Q1-Pad2): track 20.2 -> 0.00 mm, vias 1 -> 0
- net Net-(Q2-Pad2): track 16.7 -> 0.00 mm, vias 1 -> 0
- net Net-(D1-Pad1): track 11.6 -> 0.00 mm
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Other:
- board size 53.3 x 54.6 mm -> 83.2 x 126.3 mm
- net class Default: clearance 0.254 -> 0.2; trace_width 0.254 -> 0.25; via_dia 0.762 -> 0.6; via_drill 0.381 -> 0.4
- rule pad_to_mask_clearance: 0.0508 -> 0.2
- rule trace_clearance: 0.254 -> 0.2
- rule trace_min: 0.1524 -> 0.2
- rule via_min_drill: 0.3302 -> 0.3
- rule via_min_size: 0.6858 -> 0.4
- board text added: "LM324N_Line_Follower v.01 AJ Dahal- SP2020 Hunter Engineering 04"
- board text removed: "LM324N_Line_Follower v01 Ajaya Dahal-AJ- SP2020 Electrical Engineering Co-Op Electronics Plant, 04 Hunter Engineering"
