File: Projects/KiCad/FINAL lm324m_Line/lm324m_Line/New_Schematics/new schematics.kicad_pcb (KiCad board)
At the start: 2 copper layers, 87.2 x 74.6 mm, 28 parts, among them J1 CONN_01X03_MALE, J2 CONN_01X03_MALE, J3 CONN_01X03_MALE, J4 CONN_01X03_MALE, J5 Screw_Terminal_1x02, K1 EC2-5NU, K2 EC2-5NU, Q1 2N3904, Q2 2N3904, U1 lm324, U2 Tran AMS1117-5.0

Commit message: renewed
renewed
Parts:
- removed F1+: FUSE, lm324m_Line:C320C
- removed G***: , lm324m_Line:logo
- added ?: , Mounting_Holes:MountingHole_3.2mm_M3, F.Cu at (120.2, 169.9)
- added ?: , Mounting_Holes:MountingHole_3.2mm_M3, F.Cu at (45.1, 169.5)
- added ?: , Mounting_Holes:MountingHole_3.2mm_M3, F.Cu at (120.1, 64.8)
- added ?: , Mounting_Holes:MountingHole_3.2mm_M3, F.Cu at (45.3, 65.6)
- added F1: , lm324m_Line:C320C, F.Cu at (46.1, 83.0)
- added J6: , Connector_PinHeader_2.54mm new:PinHeader_1x03_P2.54mm_Vertical, F.Cu at (52.0, 69.0)
- added J7: 9V+, Connector_PinHeader_2.54mm new:PinHeader_1x02_P2.54mm_Vertical, F.Cu at (52.0, 83.0)
- added J8: , Connector_PinHeader_2.54mm new:PinHeader_1x04_P2.54mm_Vertical, F.Cu at (53.0, 155.7)
- added TB1: ARDUINO_NANO, SHIELD_ARDUINO_NANO, F.Cu at (72.0, 113.0)
- added U3: L293D, DIP880W50P254L2000H510Q16, F.Cu at (104.0, 128.2)
- D1, D2: value 1N4001 -> (none); footprint Diodes_THT:D_T-1_P12.70mm_Horizontal -> Diode_THT:D_DO-15_P15.24mm_Horizontal
- D3, D4: footprint LEDs:LED_D3.0mm -> LEDs:LED_D4.0mm
- J1, J2, J3, J4: value CONN_01X03_MALE -> (none); footprint Connectors_Molex:Molex_KK-41791-03_03x3.96mm_Straight -> Connector_PinHeader_2.54mm new:PinHeader_1x03_P2.54mm_Vertical
- J5: value Screw_Terminal_1x02 -> (none); footprint 2 pin male connector:2_pin_male_connector -> Connector_PinHeader_2.54mm new:PinHeader_1x02_P2.54mm_Vertical
- K1, K2: value EC2-5NU -> (none)
- Q1, Q2: value 2N3904 -> (none); footprint 2N3904:TO92127P495H495-3 -> TO_SOT_Packages_THT:TO-92_Inline_Wide
- R1, R2: footprint pot:TRIM_3266W-1-103LF -> Potentiometers:Potentiometer_Trimmer_ACP_CA6v_Horizontal
- R4: value 270 -> (none)
- U2: value Tran AMS1117-5.0 -> AMS1117-5.0
- moved R10 95.9 mm to (64.4, 69.0), turned to 0 degrees
- moved R3 72.7 mm to (64.2, 162.0), turned to 0 degrees
- moved J3 61.5 mm to (60.0, 129.0)
- moved J5 59.1 mm to (52.0, 90.0), turned to 90 degrees
- moved R4 58.8 mm to (89.7, 162.0)
- moved D1 51.7 mm to (70.0, 153.0), turned to 0 degrees
- moved K1 48.4 mm to (85.0, 144.0), turned to 90 degrees
- moved R8 45.5 mm to (115.0, 88.5)
- moved J4 45.4 mm to (60.0, 141.0)
- moved U2 45.0 mm to (51.8, 97.0)
- moved D3 43.2 mm to (52.0, 129.6), turned to 0 degrees
- moved R9 42.7 mm to (110.3, 69.0), turned to 180 degrees
- moved U1 39.5 mm to (104.0, 88.1), turned to 270 degrees
- moved J2 39.2 mm to (53.0, 162.0)
- moved Q2 35.9 mm to (72.0, 146.6), turned to 90 degrees
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Connections:
- D1 pad 1: Net-(D1-Pad1) -> V+
- D2 pad 1: Net-(D2-Pad1) -> V+
- J3 pad 1: Net-(J3-Pad1) -> Motor1a
- J3 pad 2: Net-(J3-Pad2) -> Motor1b
- J3 pad 3: OutputPIN1 -> (no net)
- J4 pad 1: Net-(J4-Pad1) -> Motor2a
- J4 pad 2: Net-(J4-Pad2) -> Motor2b
- J4 pad 3: OutputPIN4 -> (no net)
- K1 pad 1: Net-(D1-Pad1) -> V+
- K1 pad 10: Net-(K1-Pad10) -> (no net)
- K1 pad 3: Net-(K1-Pad3) -> (no net)
- K1 pad 4: Net-(J3-Pad1) -> Motor2a
- K1 pad 5: Net-(J3-Pad2) -> Motor2b
- K1 pad 8: Net-(K1-Pad8) -> (no net)
- K1 pad 9: Net-(K1-Pad9) -> (no net)
- K2 pad 1: Net-(D2-Pad1) -> V+
- K2 pad 10: Net-(K2-Pad10) -> (no net)
- K2 pad 3: Net-(K2-Pad3) -> (no net)
- K2 pad 4: Net-(J4-Pad1) -> Motor1a
- K2 pad 5: Net-(J4-Pad2) -> Motor1b
- K2 pad 8: Net-(K2-Pad8) -> (no net)
- K2 pad 9: Net-(K2-Pad9) -> (no net)
- U1 pad 10: Net-(U1-Pad10) -> (no net)
- U1 pad 5: Net-(U1-Pad5) -> (no net)
- U1 pad 6: Net-(U1-Pad6) -> (no net)
- U1 pad 7: Net-(U1-Pad7) -> (no net)
- U1 pad 8: Net-(U1-Pad8) -> (no net)
- U1 pad 9: Net-(U1-Pad9) -> (no net)
- U2 pad 2: V+ -> Net-(J6-Pad2)
Routing:
- net GND: track 154.6 -> 0.00 mm, vias 1 -> 0
- net Input4-: track 119.7 -> 0.00 mm, vias 4 -> 0
- net V+: track 114.8 -> 0.00 mm, vias 5 -> 0
- net OutputPIN1: track 84.3 -> 0.00 mm, vias 4 -> 0
- net Net-(D3-Pad2): track 83.8 -> 0.00 mm, vias 6 -> 0
- net Net-(J3-Pad1): track 68.1 -> 0.00 mm, vias 8 -> 0
- net Net-(J3-Pad2): track 62.4 -> 0.00 mm, vias 4 -> 0
- net OutputPIN4: track 56.4 -> 0.00 mm
- net +9V: track 53.8 -> 0.00 mm
- net Net-(J2-Pad2): track 52.0 -> 0.00 mm, vias 1 -> 0
- net Input1-: track 46.1 -> 0.00 mm, vias 1 -> 0
- net Net-(Q1-Pad2): track 44.4 -> 0.00 mm, vias 2 -> 0
- net Net-(D4-Pad2): track 34.0 -> 0.00 mm, vias 3 -> 0
- net Net-(Q2-Pad2): track 32.6 -> 0.00 mm, vias 1 -> 0
- net Net-(J4-Pad1): track 29.5 -> 0.00 mm
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Other:
- board size 87.2 x 74.6 mm -> 83.2 x 126.3 mm
- board text added: "LM324N_Line_Follower v.01 AJ Dahal- SP2020 Hunter Engineering 04"
- board text removed: "+"
- board text removed: "Ajaya Dahal-AJ Co-Op MSSTATE Hunter Engineering, Electronics Plant 04, Raymond, MS"
- board text removed: "In1"
- board text removed: "In4"
- board text removed: "O1"
- board text removed: "O4"
