File: Projects/KiCad/FINAL lm324m_Line/lm324m_Line/New_Schematics/new schematics.sch (KiCad schematic (older format))
At the start: 32 parts, among them J1 CONN_01X03_MALE (DATA) PIN 3, J2 CONN_01X03_MALE (DATA) PIN 3, J3 CONN_01X03_MALE, J4 CONN_01X03_MALE, J5 Screw_Terminal_1x02, J6 CONN_01X03_MALE 1-Ard, J7 9V+, J8 CONN Arduino Backup Motor dri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, K1 EC2-5NU, K2 EC2-5NU, Q1 2N3904, Q2 2N3904, U1 lm324, U2 AMS1117-5.0, U3 L293D

Commit message: renewed
renewed
Parts:
- 0.1uf1: footprint Capacitors_THT:CP_Radial_D10.0mm_P5.00mm -> Capacitors_THT:CP_Radial_D4.0mm_P1.50mm
- D1, D2: footprint Diodes_THT:D_T-1_P12.70mm_Horizontal -> Diode_THT:D_DO-15_P15.24mm_Horizontal
- D3, D4: footprint LEDs:LED_D3.0mm -> LEDs:LED_D4.0mm
- J1, J2, J3, J4, J6: footprint Connectors_Molex:Molex_KK-41791-03_03x3.96mm_Straight -> Connector_PinHeader_2.54mm new:PinHeader_1x03_P2.54mm_Vertical
- J5, J7: footprint 2 pin male connector:2_pin_male_connector -> Connector_PinHeader_2.54mm new:PinHeader_1x02_P2.54mm_Vertical
- J8: footprint Connectors_Molex:Molex_KK-41791-04_04x3.96mm_Straight -> Connector_PinHeader_2.54mm new:PinHeader_1x04_P2.54mm_Vertical
- Q1, Q2: footprint 2N3904:TO92127P495H495-3 -> TO_SOT_Packages_THT:TO-92_Inline_Wide
- R1, R2: footprint pot:TRIM_3266W-1-103LF -> Potentiometers:Potentiometer_Trimmer_ACP_CA6v_Horizontal
Connections:
- net 5V+ard: now also TB1.30 (VIN); no longer TB1.27 (+5V)
Changed lines of the file:
@@
 F 0 "J5" H 11050 1400 50  0000 C TNN
 F 1 "Screw_Terminal_1x02" V 10900 950 50  0000 C TNN
-F 2 "2 pin male connector:2_pin_male_connector" H 11050 925 50  0001 C CNN
+F 2 "Connector_PinHeader_2.54mm new:PinHeader_1x02_P2.54mm_Vertical" H 11050 925 50  0001 C CNN
 F 3 "" H 11025 1150 50  0001 C CNN
 	1    11050 1150
@@
 F 0 "Q1" H 3400 7250 50  0000 L BNN
 F 1 "2N3904" H 3400 6650 50  0000 L BNN
-F 2 "2N3904:TO92127P495H495-3" H 3800 6950 50  0001 L BNN
+F 2 "TO_SOT_Packages_THT:TO-92_Inline_Wide" H 3800 6950 50  0001 L BNN
 F 3 "February 2003" H 3800 6950 50  0001 L BNN
 F 4 "STMicroelectronics" H 3800 6950 50  0001 L BNN "Field4"
@@
 F 0 "D3" H 4400 6750 50  0000 C CNN
 F 1 "LED" H 4400 6550 50  0000 C CNN
-F 2 "LEDs:LED_D3.0mm" H 4400 6650 50  0001 C CNN
+F 2 "LEDs:LED_D4.0mm" H 4400 6650 50  0001 C CNN
 F 3 "" H 4400 6650 50  0001 C CNN
 	1    4400 6650
@@
 F 0 "D1" H 3100 6550 50  0000 C CNN
 F 1 "1N4001" H 3100 6350 50  0000 C CNN
-F 2 "Diodes_THT:D_T-1_P12.70mm_Horizontal" H 3100 6275 50  0001 C CNN
+F 2 "Diode_THT:D_DO-15_P15.24mm_Horizontal" H 3100 6275 50  0001 C CNN
 F 3 "" H 3100 6450 50  0001 C CNN
 	1    3100 6450
@@
 F 0 "R2" V 3350 4150 50  0000 L CNN
 F 1 "10k" V 3150 4200 50  0000 L CNN
-F 2 "pot:TRIM_3266W-1-103LF" V 3180 4250 50  0001 C CNN
+F 2 "Potentiometers:Potentiometer_Trimmer_ACP_CA6v_Horizontal" V 3180 4250 50  0001 C CNN
 F 3 "" H 3250 4250 50  0001 C CNN
 	1    3250 4250
@@
 F 0 "J3" H 8200 6425 50  0000 C CNN
 F 1 "CONN_01X03_MALE" H 8225 5875 50  0000 C CNN
-F 2 "Connectors_Molex:Molex_KK-41791-03_03x3.96mm_Straight" H 8200 6350 50  0001 C CNN
+F 2 "Connector_PinHeader_2.54mm new:PinHeader_1x03_P2.54mm_Vertical" H 8200 6350 50  0001 C CNN
 F 3 "" H 8200 6350 50  0001 C CNN
 	1    8200 6150
@@
 F 0 "Q2" H 3450 1550 50  0000 L BNN
 F 1 "2N3904" H 3450 950 50  0000 L BNN
-F 2 "2N3904:TO92127P495H495-3" H 3850 1250 50  0001 L BNN
+F 2 "TO_SOT_Packages_THT:TO-92_Inline_Wide" H 3850 1250 50  0001 L BNN
 F 3 "February 2003" H 3850 1250 50  0001 L BNN
 F 4 "STMicroelectronics" H 3850 1250 50  0001 L BNN "Field4"
@@
 F 0 "D4" H 4450 1050 50  0000 C CNN
 F 1 "LED" H 4450 850 50  0000 C CNN
-F 2 "LEDs:LED_D3.0mm" H 4450 950 50  0001 C CNN
+F 2 "LEDs:LED_D4.0mm" H 4450 950 50  0001 C CNN
 F 3 "" H 4450 950 50  0001 C CNN
 	1    4450 950
@@
 F 0 "D2" H 3150 850 50  0000 C CNN
 F 1 "1N4001" H 3150 650 50  0000 C CNN
-F 2 "Diodes_THT:D_T-1_P12.70mm_Horizontal" H 3150 575 50  0001 C CNN
+F 2 "Diode_THT:D_DO-15_P15.24mm_Horizontal" H 3150 575 50  0001 C CNN
 F 3 "" H 3150 750 50  0001 C CNN
 	1    3150 750
@@
 F 0 "J4" H 9150 6425 50  0000 C CNN
 F 1 "CONN_01X03_MALE" H 9175 5875 50  0000 C CNN
-F 2 "Connectors_Molex:Molex_KK-41791-03_03x3.96mm_Straight" H 9150 6350 50  0001 C CNN
+F 2 "Connector_PinHeader_2.54mm new:PinHeader_1x03_P2.54mm_Vertical" H 9150 6350 50  0001 C CNN
 F 3 "" H 9150 6350 50  0001 C CNN
 	1    9150 6150
@@
 F 0 "J2" H 2200 4525 50  0000 C CNN
 F 1 "CONN_01X03_MALE (DATA) PIN 3" H 2200 3900 50  0000 C CNN
-F 2 "Connectors_Molex:Molex_KK-41791-03_03x3.96mm_Straight" H 2200 4450 50  0001 C CNN
+F 2 "Connector_PinHeader_2.54mm new:PinHeader_1x03_P2.54mm_Vertical" H 2200 4450 50  0001 C CNN
 F 3 "" H 2200 4450 50  0001 C CNN
 	1    2200 4250
@@
 F 0 "0.1uf1" H 10675 1700 50  0000 L CNN
 F 1 "CP" H 10675 1500 50  0000 L CNN
-F 2 "Capacitors_THT:CP_Radial_D10.0mm_P5.00mm" H 10688 1450 50  0001 C CNN
+F 2 "Capacitors_THT:CP_Radial_D4.0mm_P1.50mm" H 10688 1450 50  0001 C CNN
 F 3 "" H 10650 1600 50  0001 C CNN
 	1    10650 1600
@@
 F 0 "R1" V 3350 3000 50  0000 L CNN
 F 1 "10k" V 3150 3050 50  0000 L CNN
-F 2 "pot:TRIM_3266W-1-103LF" V 3180 3100 50  0001 C CNN
+F 2 "Potentiometers:Potentiometer_Trimmer_ACP_CA6v_Horizontal" V 3180 3100 50  0001 C CNN
 F 3 "" H 3250 3100 50  0001 C CNN
 	1    3250 3100
@@
 F 0 "J1" H 2200 3375 50  0000 C CNN
 F 1 "CONN_01X03_MALE (DATA) PIN 3" H 2250 2750 50  0000 C CNN
-F 2 "Connectors_Molex:Molex_KK-41791-03_03x3.96mm_Straight" H 2200 3300 50  0001 C CNN
+F 2 "Connector_PinHeader_2.54mm new:PinHeader_1x03_P2.54mm_Vertical" H 2200 3300 50  0001 C CNN
 F 3 "" H 2200 3300 50  0001 C CNN
 	1    2200 3100
@@
 Text GLabel 9400 4650 3    60   Input ~ 0
 arOutputPIN4
-Text GLabel 11000 4700 3    60   Input ~ 0
+Text GLabel 10600 3250 1    60   Input ~ 0
 5V+ard
 Text GLabel 8400 4700 3    60   Input ~ 0
@@
 F 0 "J6" H 8950 2225 50  0000 C CNN
 F 1 "CONN_01X03_MALE 1-Ard" V 8800 2150 50  0000 C CNN
-F 2 "Connectors_Molex:Molex_KK-41791-03_03x3.96mm_Straight" H 8950 2150 50  0001 C CNN
+F 2 "Connector_PinHeader_2.54mm new:PinHeader_1x03_P2.54mm_Vertical" H 8950 2150 50  0001 C CNN
 F 3 "" H 8950 2150 50  0001 C CNN
 	1    8950 1950
@@
 F 0 "J7" H 10300 875 50  0000 C CNN
 F 1 "9V+" H 10100 800 50  0000 C CNN
-F 2 "2 pin male connector:2_pin_male_connector" H 10300 800 50  0001 C CNN
+F 2 "Connector_PinHeader_2.54mm new:PinHeader_1x02_P2.54mm_Vertical" H 10300 800 50  0001 C CNN
 F 3 "" H 10300 800 50  0001 C CNN
 	1    10300 700
@@
 F 0 "J8" H 10400 6475 50  0000 C CNN
 F 1 "CONN Arduino Backup Motor driver" H 10750 5700 50  0000 C CNN
-F 2 "Connectors_Molex:Molex_KK-41791-04_04x3.96mm_Straight" H 10400 6400 50  0001 C CNN
+F 2 "Connector_PinHeader_2.54mm new:PinHeader_1x04_P2.54mm_Vertical" H 10400 6400 50  0001 C CNN
 F 3 "" H 10400 6400 50  0001 C CNN
 	1    10400 6100
@@
 NoConn ~ 10800 4650
 NoConn ~ 10900 4650
-NoConn ~ 10600 3250
 NoConn ~ 10500 3250
 NoConn ~ 10300 3250
@@
 NoConn ~ 9400 3250
 NoConn ~ 9300 3250
-Connection ~ 6850 5850
 Wire Wire Line
 	10600 600  10700 600
@@
 	4400 6800 4400 6950
 Connection ~ 4400 6950
-Wire Wire Line
-	11000 4650 11000 4700
 Connection ~ 10500 3250
 Wire Wire Line
@@
 V+
 Connection ~ 2800 6550
+NoConn ~ 11000 4650
 $EndSCHEMATC
