File: Projects/KiCad/FINAL lm324m_Line/lm324m_Line/with arduino/with arduino.kicad_pcb (KiCad board)
At the start: 2 copper layers, 100.7 x 98.3 mm, 37 parts, among them J1 CONN_01X03_MALE (DATA) PIN 3, J2 CONN_01X03_MALE (DATA) PIN 3, J3 CONN_01X03_MALE, J4 CONN_01X03_MALE, J5 Screw_Terminal_1x02, J6 CONN_01X03_MALE 1-Ard, J7 9V+, J8 CONN Arduino Backup Motor dri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, K1 EC2-5NU, K2 EC2-5NU, Q1 2N3904, Q2 2N3904, U1 lm324, U2 AMS1117-5.0, U3 L293D

Commit message: renewed
renewed
Parts:
- removed G***: LOGO, lm324m_Line:logo
- ? (x4): renamed from REF**; value MountingHole_3.2mm_M3 -> (none)
- D1, D2: value 1N4001 -> (none); footprint Diodes_THT:D_T-1_P12.70mm_Horizontal -> Diode_THT:D_DO-15_P15.24mm_Horizontal
- D3, D4: footprint LEDs:LED_D3.0mm -> LEDs:LED_D4.0mm
- F1: value FUSE -> (none)
- J1, J2: value CONN_01X03_MALE (DATA) PIN 3 -> (none); footprint Connectors_Molex:Molex_KK-41791-03_03x3.96mm_Straight -> Connector_PinHeader_2.54mm new:PinHeader_1x03_P2.54mm_Vertical
- J3, J4: value CONN_01X03_MALE -> (none); footprint Connectors_Molex:Molex_KK-41791-03_03x3.96mm_Straight -> Connector_PinHeader_2.54mm new:PinHeader_1x03_P2.54mm_Vertical
- J5: value Screw_Terminal_1x02 -> (none); footprint 2 pin male connector:2_pin_male_connector -> Connector_PinHeader_2.54mm new:PinHeader_1x02_P2.54mm_Vertical
- J6: value CONN_01X03_MALE 1-Ard -> (none); footprint Connectors_Molex:Molex_KK-41791-03_03x3.96mm_Straight -> Connector_PinHeader_2.54mm new:PinHeader_1x03_P2.54mm_Vertical
- J7: footprint 2 pin male connector:2_pin_male_connector -> Connector_PinHeader_2.54mm new:PinHeader_1x02_P2.54mm_Vertical
- J8: value CONN Arduino Backup Motor driver -> (none); footprint Connectors_Molex:Molex_KK-41791-04_04x3.96mm_Straight -> Connector_PinHeader_2.54mm new:PinHeader_1x04_P2.54mm_Vertical
- K1, K2: value EC2-5NU -> (none)
- Q1, Q2: value 2N3904 -> (none); footprint 2N3904:TO92127P495H495-3 -> TO_SOT_Packages_THT:TO-92_Inline_Wide
- R1, R2: footprint pot:TRIM_3266W-1-103LF -> Potentiometers:Potentiometer_Trimmer_ACP_CA6v_Horizontal
- R4: value 270 -> (none)
- moved ? 134.3 mm to (83.8, 55.3)
- moved ? 118.6 mm to (68.8, 54.4)
- moved D4 117.6 mm to (52.0, 140.4)
- moved J3 117.5 mm to (60.0, 129.0)
- moved R10 110.3 mm to (64.4, 69.0)
- moved J5 101.9 mm to (52.0, 90.0), turned to 90 degrees
- moved J6 101.1 mm to (52.0, 69.0), turned to 90 degrees
- moved R3 100.0 mm to (64.2, 162.0)
- moved D2 98.5 mm to (90.7, 153.0), turned to 0 degrees
- moved Q1 93.3 mm to (72.0, 134.7), turned to 90 degrees
- moved F1 93.1 mm to (46.1, 83.0), turned to 180 degrees
- moved J8 91.9 mm to (53.0, 155.7), turned to 180 degrees
- moved K2 90.1 mm to (85.0, 132.0), turned to 90 degrees
- moved R4 89.4 mm to (89.7, 162.0)
- moved ? 87.1 mm to (100.6, 53.7)
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Connections:
- D1 pad 1: Net-(D1-Pad1) -> V+
- D2 pad 1: Net-(D2-Pad1) -> V+
- J3 pad 3: Net-(J3-Pad3) -> (no net)
- J4 pad 3: Net-(J4-Pad3) -> (no net)
- K1 pad 1: Net-(D1-Pad1) -> V+
- K1 pad 10: Net-(K1-Pad10) -> (no net)
- K1 pad 3: Net-(K1-Pad3) -> (no net)
- K1 pad 8: Net-(K1-Pad8) -> (no net)
- K1 pad 9: Net-(K1-Pad9) -> (no net)
- K2 pad 1: Net-(D2-Pad1) -> V+
- K2 pad 10: Net-(K2-Pad10) -> (no net)
- K2 pad 3: Net-(K2-Pad3) -> (no net)
- K2 pad 8: Net-(K2-Pad8) -> (no net)
- K2 pad 9: Net-(K2-Pad9) -> (no net)
- TB1 pad 1: Net-(TB1-Pad1) -> (no net)
- TB1 pad 11: Net-(TB1-Pad11) -> (no net)
- TB1 pad 12: Net-(TB1-Pad12) -> (no net)
- TB1 pad 13: Net-(TB1-Pad13) -> (no net)
- TB1 pad 14: Net-(TB1-Pad14) -> (no net)
- TB1 pad 15: Net-(TB1-Pad15) -> (no net)
- TB1 pad 16: Net-(TB1-Pad16) -> (no net)
- TB1 pad 17: Net-(TB1-Pad17) -> (no net)
- TB1 pad 18: Net-(TB1-Pad18) -> (no net)
- TB1 pad 19: Net-(TB1-Pad19) -> (no net)
- TB1 pad 2: Net-(TB1-Pad2) -> (no net)
- TB1 pad 20: Net-(TB1-Pad20) -> (no net)
- TB1 pad 21: Net-(TB1-Pad21) -> (no net)
- TB1 pad 22: Net-(TB1-Pad22) -> (no net)
- TB1 pad 23: Net-(TB1-Pad23) -> (no net)
- TB1 pad 24: Net-(TB1-Pad24) -> (no net)
- TB1 pad 25: Net-(TB1-Pad25) -> (no net)
- TB1 pad 26: Net-(TB1-Pad26) -> (no net)
- TB1 pad 27: 5V+ard -> (no net)
- TB1 pad 30: Net-(TB1-Pad30) -> 5V+ard
- U1 pad 10: Net-(U1-Pad10) -> (no net)
- U1 pad 5: Net-(U1-Pad5) -> (no net)
- U1 pad 6: Net-(U1-Pad6) -> (no net)
- U1 pad 7: Net-(U1-Pad7) -> (no net)
- U1 pad 8: Net-(U1-Pad8) -> (no net)
- U1 pad 9: Net-(U1-Pad9) -> (no net)
Routing:
- net GND: track 220.6 -> 0.00 mm, vias 2 -> 0
- net V+: track 127.2 -> 0.00 mm
- net Input4-: track 105.7 -> 0.00 mm, vias 7 -> 0
- net 5V+ard: track 98.6 -> 0.00 mm, vias 2 -> 0
- net 9V+: track 88.5 -> 0.00 mm, vias 4 -> 0
- net Input1-: track 88.4 -> 0.00 mm, vias 5 -> 0
- net Net-(D3-Pad2): track 87.3 -> 0.00 mm, vias 5 -> 0
- net OutputPIN1: track 79.6 -> 0.00 mm
- net Motor2b: track 78.8 -> 0.00 mm
- net Motor2a: track 76.2 -> 0.00 mm, vias 4 -> 0
- net Net-(J1-Pad2): track 66.9 -> 0.00 mm, vias 6 -> 0
- net Net-(J6-Pad2): track 65.2 -> 0.00 mm, vias 4 -> 0
- net OutputPIN4: track 61.9 -> 0.00 mm, vias 2 -> 0
- net Net-(D1-Pad2): track 61.4 -> 0.00 mm, vias 4 -> 0
- net Motor1b: track 57.7 -> 0.00 mm, vias 3 -> 0
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Other:
- board outline removed
