File: Projects/KiCad/45-1523-1 Tester/45-1523-1 Tester/45-1523-1.sch (KiCad schematic (older format))
At the start: 74 parts, among them J1.1 CONN_01X02, J1.2 CONN_01X02, J2 CONN_01X18, J3 CONN_01X06, J4 CONN_01X14, J5 CONN_01X03, J6 CONN_01X02, K1 EC2-5NU, K2 EC2-5NU, K3 G5Q-1, K4 EC2-5NU, K5 EC2-5NU, K6 EC2-5NU, K7 EC2-5NU, Q3 BC817-40, Q4 BC817-40, Q5 BC817-40, Q6 BC817-40, U1 Arduino_Nano, U2 Arduino_Nano, U3 LM7805CV, U4 LM7812CT, U6 PTN78020

Commit message: Done
End of semester
Parts:
- C1: symbol C -> Device:C
- C11, C12, C13, C14, C17: symbol 0.18UF-0603-10V-10% -> 45-1523-1-rescue:0.18UF-0603-10V-10%
- C2, C3: symbol CP1 -> Device:CP1
- C4, C5, C6, C7: symbol C_Small -> Device:C_Small
- D1: symbol D_Bridge_+-AA -> 45-1523-1-rescue:D_Bridge_+-AA
- D10, D11, D3, D4, D8, D9: symbol 1N4001 -> Diode:1N4001
- D5, D6, D7: symbol LED-GREEN0603 -> 45-1523-1-rescue:LED-GREEN0603
- F1, F2, F3, F4, F6: symbol 3413_0328_22 -> 45-1523-1-rescue:3413_0328_22
- J1.1, J1.2, J6: symbol CONN_01X02 -> conn:CONN_01X02
- J2: symbol CONN_01X18 -> conn:CONN_01X18
- J3: symbol CONN_01X06 -> conn:CONN_01X06
- J4: symbol CONN_01X14 -> conn:CONN_01X14
- J5: symbol CONN_01X03 -> conn:CONN_01X03
- K1, K2, K4, K5, K6, K7: symbol EC2-5NU -> 45-1523-1-rescue:EC2-5NU
- K3: symbol FINDER-36.11.4001 -> relays:FINDER-36.11.4001
- Q3, Q4, Q5, Q6: symbol BC817-40 -> transistors:BC817-40
- R1, R10, R11, R12, R13, R14, R15, R16, R17, R18, R19, R2, R20, R21, R22, R23, R24, R26, R3, R4, R5, R6, R9: symbol RESISTORAXIAL-0.3 -> 45-1523-1-rescue:RESISTORAXIAL-0.3
- R25: symbol RESISTOR0402 -> 45-1523-1-rescue:RESISTOR0402
- U1, U2: symbol Arduino_Nano -> 45-1523-1-rescue:Arduino_Nano
- U3, U4: symbol L7805CV -> 45-1523-1-rescue:L7805CV
- U6: symbol DIL8 -> conn:DIL8
Connections:
- wire segments 231 -> 285
